File: FeatherAdapter.brd (EAGLE design)
At the start: 160 x 100 mm, 10 parts, among them Q1 DMG3404, U1 B_SERIES_M.2EKEY_3042

Commit message: Continued schematic capture
Parts:
- added C3: 0.1uF, bschulz_passives:C0603
- added D2: LEDBLUE0603, bschulz:LED_0603
- added D3: LEDAMBER0603, bschulz:LED_0603
- added R1: 1k, bschulz_passives:R0603
- added R2, R3: 10k, bschulz_passives:R0603
- added R4, R5, R6: 4.7k, bschulz_passives:R0603
- added S1, S2: BUTTON4.5X4.5, bschulz:SWITCH_4.5MM
Connections:
- net VCC renamed N$1
- removed net VBUS: U1.16
- new net ANODE: D3.ANODE
- new net CATHODE: D3.CATHODE
- new net N$2: D2.ANODE, R1.2
- new net N$3: D1.1, R6.1
- new net N$4: D1.4, R5.1
- new net N$5: D1.3, R4.1
- net !RST: now also C3.1, R2.1, S1.1, S1.2
- net 3V3: now also D1.2, R2.2, R3.2
- net BLUE: now also R4.2
- net D+: now also U1.11
- net D-: now also U1.13
- net D7: now also R1.1
- net GND: now also C3.2, D2.CATHODE, S1.3, S1.4, S2.3, S2.4
- net GREEN: now also R5.2
- net MODE: now also R3.1, S2.1, S2.2
- net RED: now also R6.2
- net VUSB: now also U1.16
