File: FeatherAdapter.brd (EAGLE design)
At the start: 160 x 100 mm, 10 parts, among them Q1 DMG3404, U1 B_SERIES_M.2EKEY_3042

Commit message: Further schematic capture
Parts:
- added C3, C4: 1uF, bschulz_passives:C0603
- added C5, C6: 4.7uF, bschulz_passives:C0805
- added C7: 0.1uF, bschulz_passives:C0603
- added D2: LEDBLUE0603, bschulz:LED_0603
- added D3: LEDAMBER0603, bschulz:LED_0603
- added F1: (no value), bschulz:1206
- added JP1: JUMPER-SMT_2_NC_PASTE_SILK_ROUND, bschulz:SMT-JUMPER_2_NC_SILK_ROUND
- added Q2: NX2301P, bschulz:SOT23-3
- added Q4: 2N7002, bschulz:SOT23-3
- added R1: 2k, bschulz_passives:R0603
- added R11, R12, R3, R5, R6: 4.7k, bschulz_passives:R0603
- added R2, R4: 1M, bschulz_passives:R0603
- added R7, R8: 100k, bschulz_passives:R0603
- added S1, S2: BUTTON4.5X4.5, bschulz:SWITCH_4.5MM
- added U2: TLV755P3V3SOT23, bschulz:DBV0005A
- added U3: MCP73832SOT, bschulz:SOT23-5
- USB1: value USB_MICROMUSB-K152 -> USB_MICRO; device bschulz:MUSB-K152-30 -> bschulz:10118194-0001LF_10118194-0001LF_LONGER_PADS
Connections:
- removed net VBUS: U1.16
- new net EN: MS1.27, Q4.1, R2.1
- new net EN_GATE: Q2.1, Q4.3, R4.1
- new net N$1: R1.1, U3.2
- new net N$10: D3.ANODE, R12.2
- new net N$2: R1.2, U3.5
- new net N$3: C1.1, C2.1, F1.1, USB1.1
- new net N$4: D2.CATHODE, JP1.1
- new net N$5: D1.1, R3.1
- new net N$6: D1.4, R5.1
- new net N$7: D1.3, R6.1
- new net N$8: D2.ANODE, R11.1
- new net STAT: R12.1, U3.1
- net !RST: now also C7.1, MS1.1, R7.1, S2.1, S2.2
- net 3V3: now also C4.1, D1.2, MS1.2, R7.2, R8.2, U2.5
- net BAT+: now also C6.1, Q2.2, R2.2, R4.2, U3.3
- net BLUE: now also R6.2
- net D+: now also U1.11
- net D-: now also U1.13
- net D7: now also R11.2
- net GND: now also C3.2, C4.2, C5.2, C6.2, C7.2, D3.CATHODE, JP1.2, Q4.2, S1.3, S1.4, S2.3, S2.4, U2.2
- net GREEN: now also R5.2
- net MODE: now also MS1.3, R8.1, S1.1, S1.2
- net RED: now also R3.2
- net VCC: now also C3.1, MS1.28, Q2.3, U2.1, U2.3
- net VUSB: now also C5.1, F1.2, MS1.26, U1.16, U3.4; no longer C1.1, C2.1, USB1.1

Commit message: Board component placement
Parts:
- C7: device bschulz_passives:C0603 -> bschulz_passives:C0402
- R1, R11, R12, R2, R3, R4, R5, R6, R7, R8: device bschulz_passives:R0603 -> bschulz_passives:R0402
- moved R11 179.2 mm to (20.3, 64.1), turned to 180 degrees
- moved R12 179.2 mm to (16.5, 64.1), turned to 180 degrees
- moved D3 171.5 mm to (16.5, 65.4), turned to 180 degrees
- moved D2 171.0 mm to (20.3, 65.4)
- moved JP1 169.4 mm to (17.8, 62.2), flipped to the bottom
- moved C7 161.5 mm to (29.6, 52.1), turned to 270 degrees
- moved R7 152.6 mm to (25.4, 48.9), turned to 180 degrees
- moved S2 152.3 mm to (25.4, 52.1)
- moved R8 144.9 mm to (5.08, 48.9)
- moved S1 138.0 mm to (5.08, 52.1), turned to 180 degrees
- moved R4 133.5 mm to (20.3, 52.1), turned to 180 degrees
- moved Q4 129.6 mm to (20.3, 54.4), turned to 90 degrees
- moved R2 126.5 mm to (20.3, 50.8), turned to 180 degrees
- moved F1 124.1 mm to (12.4, 64.8)
- moved Q2 121.0 mm to (17.1, 56.5), turned to 90 degrees
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Connections:
- removed net N$1: R1.1, U3.2
- net BAT+: now also R12.1
- net GND: now also R1.1, U3.2; no longer D3.CATHODE
- net STAT: now also D3.CATHODE; no longer R12.1
Other:
- board size 160 x 100 mm -> 30.5 x 66.2 mm

Commit message: Initial layout
Parts:
- moved D3 8.39 mm to (11.7, 58.5), turned to 90 degrees
- moved R6 3.43 mm to (2.54, 4.19)
- moved R11 2.67 mm to (17.9, 65.3)
- moved R3 1.40 mm to (2.54, 6.48)
- moved D2 1.05 mm to (20.1, 64.4), turned to 90 degrees
- moved R5 1.02 mm to (2.54, 5.33)
- moved R10 0.92 mm to (5.21, 59.1), turned to 0 degrees
- moved R9 0.74 mm to (5.21, 57.9), turned to 0 degrees
- moved C5 0.25 mm to (14.5, 62.5)
- moved J2 0.13 mm to (26.8, 61.0)
- turned C7 to 90 degrees
- turned S2 to 180 degrees
Connections:
- net D+ renamed D_P
- net D- renamed D_N
Routing:
- net GND: track 0.00 -> 153.2 mm, vias 0 -> 10
- net VUSB: track 0.00 -> 132.6 mm, vias 0 -> 3
- net VCC: track 0.00 -> 102.9 mm, vias 0 -> 1
- net 3V3: track 0.00 -> 81.0 mm, vias 0 -> 3
- net D7: track 0.00 -> 77.2 mm, vias 0 -> 2
- net D_N: track 0.00 -> 71.5 mm
- net D_P: track 0.00 -> 70.3 mm
- net !RST: track 0.00 -> 61.3 mm, vias 0 -> 2
- net MODE: track 0.00 -> 60.6 mm, vias 0 -> 3
- net N$7: track 0.00 -> 59.5 mm, vias 0 -> 2
- net N$5: track 0.00 -> 57.6 mm, vias 0 -> 2
- net N$6: track 0.00 -> 56.5 mm, vias 0 -> 2
- net SCL: track 0.00 -> 48.3 mm, vias 0 -> 1
- net EN: track 0.00 -> 46.8 mm, vias 0 -> 1
- net SDA: track 0.00 -> 46.1 mm, vias 0 -> 1
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- added copper zone on layer 1, net GND
- added copper zone on layer 16, net GND
Other:
- outline, holes or cut-outs redrawn
- board text added: "+"
- board text added: "-"
- board text added: "Breakout-Particle-SoM FeatherAdapter v0.0 Bobby Schulz"
- board text added: "CHG"
- board text added: "D7"
- board text added: "J1"
- board text added: "J2"
- board text added: "J3"
- board text added: "MODE"
- board text added: "RESET"
