File: FeatherAdapter.sch (EAGLE design)
At the start: 10 parts, among them Q1 DMG3404, U1 B_SERIES_M.2EKEY_3042

Commit message: Continued schematic capture
Parts:
- added C3: 0.1uF, bschulz_passives:C-EU0.1UFC0603
- added D2: LEDBLUE0603, bschulz:LEDBLUE0603
- added D3: LEDAMBER0603, bschulz:LEDAMBER0603
- added R1: 1k, bschulz_passives:R-EU_1KR0603
- added R2, R3: 10k, bschulz_passives:R-EU_10KR0603
- added R4, R5, R6: 4.7k, bschulz_passives:R-EU_4.7KR0603
- added S1, S2: BUTTON4.5X4.5, bschulz:BUTTON4.5X4.5
Connections:
- new net 3V3: D1.ANODE, R2.2, R3.2, U1U1.3V3@10, U1U1.3V3@12
- new net N$1: U1U1.VCC@2, U1U1.VCC@4, U1U1.VCC@6, U1U1.VCC@8
- new net N$2: D2.ANODE, R1.2
- new net N$3: D1.RED_CATH, R6.1
- new net N$4: D1.GREEN_CATH, R5.1
- new net N$5: D1.BLUE_CATH, R4.1
- net !RST: now also C3.1, R2.1, S1.1, S1.2
- net BLUE: now also R4.2
- net D+: now also U1U1.USB_P
- net D-: now also U1U1.USB_N
- net D7: now also R1.1
- net GND: now also C3.2, D2.CATHODE, S1.3, S1.4, S2.3, S2.4, U1U1.GND@76, U1U1.GND@77
- net GREEN: now also R5.2
- net MODE: now also R3.1, S2.1, S2.2
- net RED: now also R6.2
- net VUSB: now also U1U1.VBUS
Other:
- note added: "FUSE?"
- moved on the sheet: D1
