File: FeatherAdapter.sch (EAGLE design)
At the start: 10 parts, among them Q1 DMG3404, U1 B_SERIES_M.2EKEY_3042

Commit message: Further schematic capture
Parts:
- added C3, C4: 1uF, bschulz_passives:C-EU1UFC0603
- added C5, C6: 4.7uF, bschulz_passives:C-EU4.7UFC0805
- added C7: 0.1uF, bschulz_passives:C-EU0.1UFC0603
- added D2: LEDBLUE0603, bschulz:LEDBLUE0603
- added D3: LEDAMBER0603, bschulz:LEDAMBER0603
- added F1: (no value), bschulz:PPTC1.5A
- added JP1: JUMPER-SMT_2_NC_PASTE_SILK_ROUND, bschulz:JUMPER-SMT_2_NC_PASTE_SILK_ROUND
- added Q2: NX2301P, bschulz:MOSFET-PCH-NX2301P
- added Q4: 2N7002, bschulz:MOSFET-NCH-2N7002P
- added R1: 2k, bschulz_passives:R-EU_2KR0603
- added R11, R12, R3, R5, R6: 4.7k, bschulz_passives:R-EU_4.7KR0603
- added R2, R4: 1M, bschulz_passives:R-EU_1MR0603
- added R7, R8: 100k, bschulz_passives:R-EU_100KR0603
- added S1, S2: BUTTON4.5X4.5, bschulz:BUTTON4.5X4.5
- added U2: TLV755P3V3SOT23, bschulz:TLV755P3V3SOT23
- added U3: MCP73832SOT, bschulz:MCP73832SOT
- USB1: value USB_MICROMUSB-K152 -> USB_MICRO; device bschulz:USB_MICROMUSB-K152 -> bschulz:USB_MICRO
Connections:
- new net 3V3: C4.1, D1.ANODE, MS1.3V, R7.2, R8.2, U1U1.3V3@10, U1U1.3V3@12, U2.VOUT
- new net EN: MS1.EN, Q4.G, R2.1
- new net EN_GATE: Q2.G, Q4.D, R4.1
- new net N$1: R1.1, U3.VSS
- new net N$10: D3.ANODE, R12.2
- new net N$2: R1.2, U3.PROG
- new net N$3: C1.1, C2.1, F1.1, USB1.VDD
- new net N$4: D2.CATHODE, JP1.1
- new net N$5: D1.RED_CATH, R3.1
- new net N$6: D1.GREEN_CATH, R5.1
- new net N$7: D1.BLUE_CATH, R6.1
- new net N$8: D2.ANODE, R11.1
- new net STAT: R12.1, U3.STAT
- new net VCC: C3.1, MS1.VBAT, Q2.D, U1U1.VCC@2, U1U1.VCC@4, U1U1.VCC@6, U1U1.VCC@8, U2.EN, U2.VIN
- net !RST: now also C7.1, MS1.!RESET, R7.1, S2.1, S2.2
- net BAT+: now also C6.1, Q2.S, R2.2, R4.2, U3.VBAT
- net BLUE: now also R6.2
- net D+: now also U1U1.USB_P
- net D-: now also U1U1.USB_N
- net D7: now also R11.2
- net GND: now also C3.2, C4.2, C5.2, C6.2, C7.2, D3.CATHODE, JP1.2, Q4.S, S1.3, S1.4, S2.3, S2.4, U1U1.GND@76, U1U1.GND@77, U2.GND
- net GREEN: now also R5.2
- net MODE: now also MS1.AREF, R8.1, S1.1, S1.2
- net RED: now also R3.2
- net VUSB: now also C5.1, F1.2, MS1.USB, U1U1.VBUS, U3.VDD; no longer C1.1, C2.1, USB1.VDD
Other:
- moved on the sheet: D1

Commit message: Board component placement
Parts:
- C7: device bschulz_passives:C-EU0.1UFC0603 -> bschulz_passives:C-EU0.1UFC0402
- R1: device bschulz_passives:R-EU_2KR0603 -> bschulz_passives:R-EU_2KR0402
- R11, R12, R3, R5, R6: device bschulz_passives:R-EU_4.7KR0603 -> bschulz_passives:R-EU_4.7KR0402
- R2, R4: device bschulz_passives:R-EU_1MR0603 -> bschulz_passives:R-EU_1MR0402
- R7, R8: device bschulz_passives:R-EU_100KR0603 -> bschulz_passives:R-EU_100KR0402
Connections:
- removed net N$1: R1.1, U3.VSS
- net BAT+: now also R12.1
- net GND: now also R1.1, U3.VSS; no longer D3.CATHODE
- net STAT: now also D3.CATHODE; no longer R12.1
Changed lines of the file:
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@@
 <part name="C5" library="bschulz_passives" deviceset="C-EU" device="C0805" technology="4.7UF" value="4.7uF"/>
 <part name="C6" library="bschulz_passives" deviceset="C-EU" device="C0805" technology="4.7UF" value="4.7uF"/>
-<part name="R1" library="bschulz_passives" deviceset="R-EU_" device="R0603" technology="2K" value="2k"/>
+<part name="R1" library="bschulz_passives" deviceset="R-EU_" device="R0402" technology="2K" value="2k"/>
 <part name="GND5" library="supply1" library_urn="urn:adsk.eagle:library:371" deviceset="GND" device=""/>
 <part name="GND6" library="supply1" library_urn="urn:adsk.eagle:library:371" deviceset="GND" device=""/>
@@
 <part name="Q2" library="bschulz" deviceset="MOSFET-PCH" device="-NX2301P" value="NX2301P"/>
 <part name="Q4" library="bschulz" deviceset="MOSFET-NCH" device="-2N7002P" value="2N7002"/>
-<part name="R2" library="bschulz_passives" deviceset="R-EU_" device="R0603" technology="1M" value="1M"/>
+<part name="R2" library="bschulz_passives" deviceset="R-EU_" device="R0402" technology="1M" value="1M"/>
 <part name="GND7" library="supply1" library_urn="urn:adsk.eagle:library:371" deviceset="GND" device=""/>
-<part name="R4" library="bschulz_passives" deviceset="R-EU_" device="R0603" technology="1M" value="1M"/>
-<part name="R3" library="bschulz_passives" deviceset="R-EU_" device="R0603" technology="4.7K" value="4.7k"/>
-<part name="R5" library="bschulz_passives" deviceset="R-EU_" device="R0603" technology="4.7K" value="4.7k"/>
-<part name="R6" library="bschulz_passives" deviceset="R-EU_" device="R0603" technology="4.7K" value="4.7k"/>
+<part name="R4" library="bschulz_passives" deviceset="R-EU_" device="R0402" technology="1M" value="1M"/>
+<part name="R3" library="bschulz_passives" deviceset="R-EU_" device="R0402" technology="4.7K" value="4.7k"/>
+<part name="R5" library="bschulz_passives" deviceset="R-EU_" device="R0402" technology="4.7K" value="4.7k"/>
+<part name="R6" library="bschulz_passives" deviceset="R-EU_" device="R0402" technology="4.7K" value="4.7k"/>
 <part name="S1" library="bschulz" deviceset="BUTTON" device="4.5X4.5"/>
 <part name="S2" library="bschulz" deviceset="BUTTON" device="4.5X4.5"/>
-<part name="R7" library="bschulz_passives" deviceset="R-EU_" device="R0603" technology="100K" value="100k"/>
-<part name="R8" library="bschulz_passives" deviceset="R-EU_" device="R0603" technology="100K" value="100k"/>
-<part name="C7" library="bschulz_passives" deviceset="C-EU" device="C0603" technology="0.1UF" value="0.1uF"/>
+<part name="R7" library="bschulz_passives" deviceset="R-EU_" device="R0402" technology="100K" value="100k"/>
+<part name="R8" library="bschulz_passives" deviceset="R-EU_" device="R0402" technology="100K" value="100k"/>
+<part name="C7" library="bschulz_passives" deviceset="C-EU" device="C0402" technology="0.1UF" value="0.1uF"/>
 <part name="GND8" library="supply1" library_urn="urn:adsk.eagle:library:371" deviceset="GND" device=""/>
 <part name="GND9" library="supply1" library_urn="urn:adsk.eagle:library:371" deviceset="GND" device=""/>
@@
 <part name="JP1" library="bschulz" deviceset="JUMPER-SMT_2_NC_PASTE" device="_SILK_ROUND"/>
 <part name="GND11" library="supply1" library_urn="urn:adsk.eagle:library:371" deviceset="GND" device=""/>
-<part name="R11" library="bschulz_passives" deviceset="R-EU_" device="R0603" technology="4.7K" value="4.7k"/>
+<part name="R11" library="bschulz_passives" deviceset="R-EU_" device="R0402" technology="4.7K" value="4.7k"/>
+<part name="R12" library="bschulz_passives" deviceset="R-EU_" device="R0402" technology="4.7K" value="4.7k"/>
 <part name="GND12" library="supply1" library_urn="urn:adsk.eagle:library:371" deviceset="GND" device=""/>
-<part name="R12" library="bschulz_passives" deviceset="R-EU_" device="R0603" technology="4.7K" value="4.7k"/>
 </parts>
 <sheets>
@@
 <attribute name="VALUE" x="72.39" y="253.238" size="1.778" layer="96"/>
 </instance>
-<instance part="GND12" gate="1" x="53.34" y="233.68" smashed="yes">
-<attribute name="VALUE" x="50.8" y="231.14" size="1.778" layer="96"/>
-</instance>
 <instance part="R12" gate="G$1" x="43.18" y="256.54" smashed="yes">
 <attribute name="NAME" x="39.37" y="258.0386" size="1.778" layer="95"/>
 <attribute name="VALUE" x="39.37" y="253.238" size="1.778" layer="96"/>
+</instance>
+<instance part="GND12" gate="1" x="142.24" y="203.2" smashed="yes">
+<attribute name="VALUE" x="139.7" y="200.66" size="1.778" layer="96"/>
 </instance>
 </instances>
@@
 </segment>
 <segment>
-<pinref part="D3" gate="G$1" pin="CATHODE"/>
+<pinref part="R1" gate="G$1" pin="1"/>
+<pinref part="U3" gate="G$1" pin="VSS"/>
+<wire x1="142.24" y1="208.28" x2="139.7" y2="208.28" width="0.1524" layer="91"/>
 <pinref part="GND12" gate="1" pin="GND"/>
-<wire x1="53.34" y1="243.84" x2="53.34" y2="236.22" width="0.1524" layer="91"/>
+<wire x1="142.24" y1="205.74" x2="142.24" y2="208.28" width="0.1524" layer="91"/>
+<junction x="142.24" y="208.28"/>
 </segment>
 </net>
@@
 <wire x1="17.78" y1="195.58" x2="15.24" y2="195.58" width="0.1524" layer="91"/>
 <label x="15.24" y="195.58" size="0.8128" layer="95" rot="R180" xref="yes"/>
+</segment>
+<segment>
+<pinref part="R12" gate="G$1" pin="1"/>
+<wire x1="38.1" y1="256.54" x2="35.56" y2="256.54" width="0.1524" layer="91"/>
+<label x="35.56" y="256.54" size="0.8128" layer="95" rot="R180" xref="yes"/>
 </segment>
 </net>
@@
 </segment>
 <segment>
-<pinref part="R12" gate="G$1" pin="1"/>
-<wire x1="38.1" y1="256.54" x2="35.56" y2="256.54" width="0.1524" layer="91"/>
-<label x="35.56" y="256.54" size="0.8128" layer="95" rot="R180" xref="yes"/>
-</segment>
-</net>
-<net name="N$1" class="0">
-<segment>
-<pinref part="R1" gate="G$1" pin="1"/>
-<pinref part="U3" gate="G$1" pin="VSS"/>
-<wire x1="142.24" y1="208.28" x2="139.7" y2="208.28" width="0.1524" layer="91"/>
-</segment>
-</net>
+<pinref part="D3" gate="G$1" pin="CATHODE"/>
+<wire x1="53.34" y1="243.84" x2="53.34" y2="238.76" width="0.1524" layer="91"/>
+<wire x1="53.34" y1="238.76" x2="55.88" y2="238.76" width="0.1524" layer="91"/>
+<label x="55.88" y="238.76" size="0.8128" layer="95" xref="yes"/>
+</segment>
+</net>
