File: FeatherAdapter.sch (EAGLE design)
At the start: 35 parts, among them Q1 DMG3404, Q2 NX2301P, Q4 2N7002, U1 B_SERIES_M.2EKEY_3042, U2 TLV755P3V3SOT23, U3 MCP73832SOT

Commit message: Initial layout
Connections:
- net D+ renamed D_P
- net D- renamed D_N
Changed lines of the file:
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@@
 <class number="0" name="default" width="0" drill="0">
+</class>
+<class number="1" name="diff pairs" width="0" drill="0">
 </class>
 </classes>
@@
 </segment>
 </net>
-<net name="D+" class="0">
-<segment>
-<pinref part="R9" gate="G$1" pin="1"/>
-<wire x1="124.46" y1="132.08" x2="121.92" y2="132.08" width="0.1524" layer="91"/>
-<label x="121.92" y="132.08" size="0.8128" layer="95" rot="R180" xref="yes"/>
-</segment>
-<segment>
-<pinref part="U1" gate="U1" pin="USB_P"/>
-<wire x1="40.64" y1="114.3" x2="38.1" y2="114.3" width="0.1524" layer="91"/>
-<label x="38.1" y="114.3" size="0.8128" layer="95" rot="R180" xref="yes"/>
-</segment>
-</net>
-<net name="D-" class="0">
-<segment>
-<pinref part="R10" gate="G$1" pin="1"/>
-<wire x1="124.46" y1="124.46" x2="121.92" y2="124.46" width="0.1524" layer="91"/>
-<label x="121.92" y="124.46" size="0.8128" layer="95" rot="R180" xref="yes"/>
-</segment>
-<segment>
-<pinref part="U1" gate="U1" pin="USB_N"/>
-<wire x1="40.64" y1="111.76" x2="38.1" y2="111.76" width="0.1524" layer="91"/>
-<label x="38.1" y="111.76" size="0.8128" layer="95" rot="R180" xref="yes"/>
-</segment>
-</net>
 <net name="BAT+" class="0">
 <segment>
@@
 </segment>
 </net>
+<net name="D_N" class="1">
+<segment>
+<pinref part="U1" gate="U1" pin="USB_N"/>
+<wire x1="40.64" y1="111.76" x2="38.1" y2="111.76" width="0.1524" layer="91"/>
+<label x="38.1" y="111.76" size="0.8128" layer="95" rot="R180" xref="yes"/>
+</segment>
+<segment>
+<pinref part="R10" gate="G$1" pin="1"/>
+<wire x1="124.46" y1="124.46" x2="121.92" y2="124.46" width="0.1524" layer="91"/>
+<label x="121.92" y="124.46" size="0.8128" layer="95" rot="R180" xref="yes"/>
+</segment>
+</net>
+<net name="D_P" class="1">
+<segment>
+<pinref part="U1" gate="U1" pin="USB_P"/>
+<wire x1="40.64" y1="114.3" x2="38.1" y2="114.3" width="0.1524" layer="91"/>
+<label x="38.1" y="114.3" size="0.8128" layer="95" rot="R180" xref="yes"/>
+</segment>
+<segment>
+<pinref part="R9" gate="G$1" pin="1"/>
+<wire x1="124.46" y1="132.08" x2="121.92" y2="132.08" width="0.1524" layer="91"/>
+<label x="121.92" y="132.08" size="0.8128" layer="95" rot="R180" xref="yes"/>
+</segment>
+</net>
